File: Power/CDR_PCB/CDR_PCB.kicad_pcb (KiCad board)
At the start: 2 copper layers, 0 parts

Commit message: Wed 04/03
Other:
- board outline added: 161.5 x 80 mm
Changed lines of the file:
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@@
 	(net 0 "")
 	(gr_rect
-		(start 118 50)
-		(end 198 130)
+		(start 170.5 39)
+		(end 250.5 119)
 		(stroke
-			(width 0.2)
+			(width 0.05)
 			(type default)
 		)
 		(fill no)
-		(layer "B.Cu")
+		(layer "Edge.Cuts")
+	)
+	(gr_rect
+		(start 89 39)
+		(end 169 119)
+		(stroke
+			(width 0.05)
+			(type default)
+		)
+		(fill no)
+		(layer "Edge.Cuts")
 	)
 	(embedded_fonts no)

Commit message: Updated PCB
Parts:
- added REF**: MountingHole_3.2mm_M3, MountingHole:MountingHole_3.2mm_M3, F.Cu at (140.0, 112.5)
- added REF**: MountingHole_3.2mm_M3, MountingHole:MountingHole_3.2mm_M3, F.Cu at (255.0, 43.0)
- added REF**: MountingHole_3.2mm_M3, MountingHole:MountingHole_3.2mm_M3, F.Cu at (255.0, 116.0)
- added REF**: PinHeader_2x25_P2.54mm_Vertical, Connector_PinHeader_2.54mm:PinHeader_2x25_P2.54mm_Vertical, F.Cu at (138.5, 45.2)
- added REF**: MountingHole_3.2mm_M3, MountingHole:MountingHole_3.2mm_M3, F.Cu at (182.0, 43.0)
- added REF**: MountingHole_3.2mm_M3, MountingHole:MountingHole_3.2mm_M3, F.Cu at (67.0, 39.5)
- added REF**: MountingHole_3.2mm_M3, MountingHole:MountingHole_3.2mm_M3, F.Cu at (67.0, 112.5)
- added REF**: MountingHole_3.2mm_M3, MountingHole:MountingHole_3.2mm_M3, F.Cu at (140.0, 39.5)
- added REF**: MountingHole_3.2mm_M3, MountingHole:MountingHole_3.2mm_M3, F.Cu at (182.0, 116.0)
- added REF**: PinHeader_2x25_P2.54mm_Vertical, Connector_PinHeader_2.54mm:PinHeader_2x25_P2.54mm_Vertical, F.Cu at (253.5, 48.8)
Other:
- board size 161.5 x 80 mm -> 195 x 83.5 mm
