File: Power/CDR_PCB/CDR_PCB.kicad_sch (KiCad schematic)
At the start: 68 parts, among them IC1 TEENSY_4.1, J1 L2596S-3.3-Breakout, J10 Transceiver header, J2 MT3608-Breakout, J4 LM2596S-5-Breakout, J5 +14Vin, J6 +14Vout, J7 MOTOR2, J8 MOTOR1, J9 Converter_GND_Lines, U1 INA226, U2 BNO055, U3 DPS310XTSA1, U4 GNSS, U5 DRV8871, U6 MICROFC-30035-SMT-TR1, U7 HTS221, U8 OPA333xxD, U9 OPA333xxD

Commit message: Finalising Sensors Schematic
Other:
- moved on the sheet: BT1, BT2, C1, C2, C3, C4, D3, D4, D5, D6, F1, F2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
