File: Power/CDR_PCB/_restore_backup_2026-08-08T18-13-06-493/CDR_PCB.kicad_sch (KiCad schematic)
At the start: 68 parts, among them IC1 TEENSY_4.1, J1 L2596S-3.3-Breakout, J10 Transceiver header, J2 MT3608-Breakout, J4 LM2596S-5-Breakout, J5 +14Vin, J6 +14Vout, J7 MOTOR2, J8 MOTOR1, J9 Converter_GND_Lines, U1 INA226, U2 BNO055, U3 DPS310XTSA1, U4 GNSS, U5 DRV8871, U6 MICROFC-30035-SMT-TR1, U7 HTS221, U8 OPA333xxD, U9 OPA333xxD

Commit message: Completed CDH Board
Changed lines of the file:
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@@
 		(at 31.75 48.26)
-	)
-	(bus_entry
-		(at 67.31 161.29)
-		(size 2.54 2.54)
-		(stroke
-			(width 0)
-			(type default)
-		)
 	)
 	(wire
