File: Power/Final_PCB/Sensors/Sensors.kicad_pcb (KiCad board)
At the start: 4 copper layers, 85 x 85 mm, 24 parts, among them J1 Left_Header, J2 Right_Header, J3 MICROFC_Board, U1 GNSS, U2 2472, U3 OPA333xxD, U4 OPA333xxD, U5 OPA333xxD

Commit message: Minor value changes
Parts:
- U2: value 2472 -> BNO055

Commit message: PCB Tweaks
Connections:
- R1 pad 1: +3V3 -> 3V3
- R2 pad 1: +3V3 -> 3V3
- U3 pad 7: +3V3 -> 3V3
- U4 pad 7: +3V3 -> 3V3
- U5 pad 7: +3V3 -> 3V3
Routing:
- net +3V3: track 112.5 -> 20.6 mm
Changed lines of the file:
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@@
 			(layers "*.Cu" "*.Mask")
 			(remove_unused_layers no)
-			(net "+3V3")
+			(net "3V3")
 			(pintype "passive")
 		)
@@
 			(layers "*.Cu" "*.Mask")
 			(remove_unused_layers no)
-			(net "+3V3")
+			(net "3V3")
 			(pintype "passive")
 		)
@@
 			(layers "F.Cu" "F.Mask" "F.Paste")
 			(roundrect_rratio 0.25)
-			(net "+3V3")
+			(net "3V3")
 			(pinfunction "V+_7")
 			(pintype "power_in")
@@
 			(layers "F.Cu" "F.Mask" "F.Paste")
 			(roundrect_rratio 0.25)
-			(net "+3V3")
+			(net "3V3")
 			(pinfunction "V+_7")
 			(pintype "power_in")
@@
 			(layers "F.Cu" "F.Mask" "F.Paste")
 			(roundrect_rratio 0.25)
-			(net "+3V3")
+			(net "3V3")
 			(pinfunction "V+_7")
 			(pintype "power_in")
@@
 	)
 	(segment
-		(start 126.15 76.39)
-		(end 126.15 78.27)
-		(width 0.2)
-		(layer "F.Cu")
-		(net "+3V3")
-	)
-	(segment
-		(start 106.31 119.64)
-		(end 110 123.33)
-		(width 0.2)
-		(layer "F.Cu")
-		(net "+3V3")
-	)
-	(segment
-		(start 110.62 89.19)
-		(end 110.62 88.613)
-		(width 0.2)
-		(layer "F.Cu")
-		(net "+3V3")
-	)
-	(segment
 		(start 111.4785 88.613)
 		(end 110.62 88.613)
@@
 	)
 	(segment
-		(start 115.12 123.135)
-		(end 114.925 123.33)
-		(width 0.2)
-		(layer "F.Cu")
-		(net "+3V3")
-	)
-	(segment
-		(start 95.15 123.33)
-		(end 94.55 122.73)
-		(width 0.2)
-		(layer "F.Cu")
-		(net "+3V3")
-	)
-	(segment
 		(start 123.7015 76.39)
 		(end 111.4785 88.613)
@@
 		(width 0.2)
 		(layer "F.Cu")
-		(net "+3V3")
-	)
-	(segment
-		(start 126.15 78.27)
-		(end 128.38 80.5)
-		(width 0.2)
-		(layer "F.Cu")
-		(net "+3V3")
-	)
-	(segment
-		(start 121.085552 123.735)
-		(end 115.72 123.735)
-		(width 0.2)
-		(layer "F.Cu")
-		(net "+3V3")
-	)
-	(segment
-		(start 141.875 123.965)
-		(end 121.315552 123.965)
-		(width 0.2)
-		(layer "F.Cu")
-		(net "+3V3")
-	)
-	(segment
-		(start 106.31 93.5)
-		(end 106.31 119.64)
-		(width 0.2)
-		(layer "F.Cu")
-		(net "+3V3")
-	)
-	(segment
-		(start 142.475 123.365)
-		(end 141.875 123.965)
-		(width 0.2)
-		(layer "F.Cu")
-		(net "+3V3")
-	)
-	(segment
-		(start 110 123.33)
-		(end 95.15 123.33)
-		(width 0.2)
-		(layer "F.Cu")
-		(net "+3V3")
-	)
-	(segment
-		(start 115.72 123.735)
-		(end 115.12 123.135)
-		(width 0.2)
-		(layer "F.Cu")
-		(net "+3V3")
-	)
-	(segment
-		(start 106.31 93.5)
-		(end 110.62 89.19)
-		(width 0.2)
-		(layer "F.Cu")
-		(net "+3V3")
-	)
-	(segment
-		(start 114.925 123.33)
-		(end 110 123.33)
-		(width 0.2)
-		(layer "F.Cu")
-		(net "+3V3")
-	)
-	(segment
-		(start 121.315552 123.965)
-		(end 121.085552 123.735)
-		(width 0.2)
-		(layer "F.Cu")
