File: Power/Final_PCB/Sensors/Sensors.kicad_sch (KiCad schematic)
At the start: 0 parts

Commit message: Finalising Sensors Schematic
Parts:
- added C1, C2, C3: 10pF, Capacitor_THT:C_Disc_D3.0mm_W1.6mm_P2.50mm, symbol Device:C
- added D1: S1223, Connector_PinHeader_2.54mm:PinHeader_1x02_P2.54mm_Horizontal, symbol Device:D_Photo
- added D2: BPW34, Connector_PinHeader_2.54mm:PinHeader_1x02_P2.54mm_Horizontal, symbol Device:D_Photo
- added J1: Left_Header, Connector_PinHeader_2.54mm:PinHeader_2x25_P2.54mm_Vertical, symbol Connector_Generic:Conn_02x25_Counter_Clockwise
- added J2: Right_Header, Connector_PinHeader_2.54mm:PinHeader_2x25_P2.54mm_Vertical, symbol Connector_Generic:Conn_02x25_Counter_Clockwise
- added J3: MICROFC_Board, symbol Connector:Screw_Terminal_01x02
- added R1, R2: 10K, Resistor_THT:R_Axial_DIN0207_L6.3mm_D2.5mm_P7.62mm_Horizontal, symbol Device:R
- added R3, R4, R5, R6: 100k, Resistor_THT:R_Axial_DIN0207_L6.3mm_D2.5mm_P7.62mm_Horizontal, symbol Device:R
- added U1: GNSS, GNSS:GNSS, symbol GNSS:746
- added U2: 2472, BNO055:BNO055, symbol BNO055:2472
- added U3, U4, U5: OPA333xxD, Package_SO:SOIC-8_3.9x4.9mm_P1.27mm, symbol Amplifier_Operational:OPA333xxD
Connections:
- new net: C2.2, D2.1 (K), R4.1, U4.2 (-)
- new net: C3.1, R6.2, U5.6
- new net: C3.2, J3.SOUT (Pin_2), R6.1, U5.2 (-)
- new net: C1.2, D1.1 (K), R3.1, U3.2 (-)
- new net: J3.VBIAS (Pin_1), R5.2
- new net +3V3: R1.1, R2.1, U1.8 (VIN), U2.1 (VIN), U3.7 (V+), U4.7 (V+), U5.7 (V+)
- new net 14.8V: J1.13 (Pin_13), J1.14 (Pin_14), J1.15 (Pin_15), J1.16 (Pin_16), J2.13 (Pin_13), J2.14 (Pin_14), J2.15 (Pin_15), J2.16 (Pin_16)
- new net 28V: J1.17 (Pin_17), J1.18 (Pin_18), J1.19 (Pin_19), J1.20 (Pin_20), J2.17 (Pin_17), J2.18 (Pin_18), J2.19 (Pin_19), J2.20 (Pin_20), R5.1
- new net 3V3: J1.5 (Pin_5), J1.6 (Pin_6), J1.7 (Pin_7), J1.8 (Pin_8), J2.5 (Pin_5), J2.6 (Pin_6), J2.7 (Pin_7), J2.8 (Pin_8)
- new net 5V: J1.10 (Pin_10), J1.11 (Pin_11), J1.12 (Pin_12), J1.9 (Pin_9), J2.10 (Pin_10), J2.11 (Pin_11), J2.12 (Pin_12), J2.9 (Pin_9)
- new net BNO_INT: J1.26 (Pin_26), J2.26 (Pin_26), U2.8 (INT)
- new net BNO_RST: J1.30 (Pin_30), J2.30 (Pin_30), R2.2, U2.6 (RST)
- new net BPW34_OUT: C2.1, J1.39 (Pin_39), J2.39 (Pin_39), R4.2, U4.6
- new net GND: D1.2 (A), D2.2 (A), J1.1 (Pin_1), J1.2 (Pin_2), J1.3 (Pin_3), J1.4 (Pin_4), J1.47 (Pin_47), J1.48 (Pin_48), J1.49 (Pin_49), J1.50 (Pin_50), J2.1 (Pin_1), J2.2 (Pin_2), J2.3 (Pin_3), J2.4 (Pin_4), J2.47 (Pin_47), J2.48 (Pin_48), J2.49 (Pin_49), J2.50 (Pin_50), U1.7 (GND), U2.10 (PS0), U2.3 (GND), U2.7 (ADR), U2.9 (PS1), U3.3 (+), U3.4 (V-), U4.3 (+), U4.4 (V-), U5.3 (+), U5.4 (V-)
- new net GNSS_EN: J1.42 (Pin_42), J2.42 (Pin_42), R1.2, U1.2 (EN)
- new net GNSS_FIX: J1.41 (Pin_41), J2.41 (Pin_41), U1.4 (FIX)
- new net GNSS_PPS: J1.40 (Pin_40), J2.40 (Pin_40), U1.9 (PPS)
- new net INA_ALERT: J1.27 (Pin_27), J2.27 (Pin_27)
- new net MICROFC: J1.28 (Pin_28), J2.28 (Pin_28)
- new net RX1: J1.44 (Pin_44), J2.44 (Pin_44), U1.5 (TX)
- new net RX2: J1.43 (Pin_43), J2.43 (Pin_43)
- new net S1223: C1.1, J1.29 (Pin_29), J2.29 (Pin_29), R3.2, U3.6
- new net SCL: J1.23 (Pin_23), J2.23 (Pin_23), U2.5 (SCL)
- new net SDA: J1.25 (Pin_25), J2.25 (Pin_25), U2.4 (SDA)
- new net TX1: J1.46 (Pin_46), J2.46 (Pin_46), U1.6 (RX)
- new net TX2: J1.45 (Pin_45), J2.45 (Pin_45)
- new net VBAT: J1.21 (Pin_21), J1.22 (Pin_22), J2.21 (Pin_21), J2.22 (Pin_22), U1.3 (VBAT)
- new net XB_RESET: J1.24 (Pin_24), J2.24 (Pin_24)
- no-connect marks 0 -> 18
Other:
- note added: "Interboard Headers"
- note added: "PhotoDiodes"
- note added: "Positional Sensors"
- title: (none) -> HYPERIONyX - Sensors Board 

Commit message: Finalised Sensors PCB
Parts:
- D1, D2: footprint Connector_PinHeader_2.54mm:PinHeader_1x02_P2.54mm_Horizontal -> Connector_PinHeader_2.54mm:PinHeader_1x02_P2.54mm_Vertical
- J3: footprint (none) -> Connector_PinHeader_2.54mm:PinHeader_1x02_P2.54mm_Vertical
Connections:
- net MICROFC: now also C3.1, R6.2, U5.6
- net at C3.2, R6.1, U5.2 (-): now also J3.2 (SOUT); no longer J3.SOUT (Pin_2)
- net at R5.2: now also J3.1 (VBIAS); no longer J3.VBIAS (Pin_1)
Changed lines of the file:
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@@
 		)
 	)
+	(global_label "MICROFC"
+		(shape input)
+		(at 157.48 101.6 0)
+		(fields_autoplaced yes)
+		(effects
+			(font
+				(size 1.27 1.27)
+			)
+			(justify left)
+		)
+		(property "Intersheetrefs" "${INTERSHEET_REFS}"
+			(at 168.7505 101.6 0)
+			(hide yes)
+			(show_name no)
+			(do_not_autoplace no)
+			(effects
+				(font
+					(size 1.27 1.27)
+				)
+				(justify left)
+			)
+		)
+	)
 	(global_label "BNO_RST"
 		(shape input)
@@
 			)
 		)
-		(property "Footprint" ""
+		(property "Footprint" "Connector_PinHeader_2.54mm:PinHeader_1x02_P2.54mm_Vertical"
 			(at 125.73 90.17 0)
 			(hide yes)
@@
 			)
 		)
-		(pin "VBIAS"
+		(pin "2"
 		)
-		(pin "SOUT"
+		(pin "1"
 		)
 		(instances
@@
 			)
 		)
-		(property "Footprint" "Connector_PinHeader_2.54mm:PinHeader_1x02_P2.54mm_Horizontal"
+		(property "Footprint" "Connector_PinHeader_2.54mm:PinHeader_1x02_P2.54mm_Vertical"
 			(at 22.86 110.49 0)
 			(hide yes)
@@
 			)
 		)
-		(property "Footprint" "Connector_PinHeader_2.54mm:PinHeader_1x02_P2.54mm_Horizontal"
+		(property "Footprint" "Connector_PinHeader_2.54mm:PinHeader_1x02_P2.54mm_Vertical"
 			(at 74.93 110.49 0)
 			(hide yes)

Commit message: Minor value changes
Parts:
- U2: value 2472 -> BNO055
Changed lines of the file:
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@@
 			)
 		)
-		(property "Value" "2472"
+		(property "Value" "BNO055"
 			(at 127 33.02 0)
 			(show_name no)

Commit message: PCB Tweaks
Connections:
- net +3V3: no longer R1.1, R2.1, U3.7 (V+), U4.7 (V+), U5.7 (V+)
- net 3V3: now also R1.1, R2.1, U3.7 (V+), U4.7 (V+), U5.7 (V+)
